File: ESP32-P4-dev-board.kicad_sch (KiCad schematic)
At the start: 172 parts, among them Q1 SS8050, Q2 SS8050, SW1 KMR221GLFS, SW2 KMR221GLFS, SW3 KMR221GLFS, SW4 KMR221GLFS, U1 TLV62569DBV, U10 AP2127K-ADJTRG1, U11 AP2127K-ADJTRG1, U12 ESP-WROOM-02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

Commit message: трассировка и проверка завершены
Parts:
- X4, X5: footprint Connector_PinSocket_2.54mm:PinSocket_1x15_P2.54mm_Vertical -> Connector_PinSocket_1.27mm:PinSocket_1x15_P1.27mm_Vertical
Connections:
- net +3.3V: now also D6.9 (K8), X5.2 (Pin_2), X5.3 (Pin_3); no longer D6.1 (K1)
- net CAM_CLK_N: now also U8.44 (CSI_CLKP); no longer U8.45 (CSI_CLKN)
- net CAM_CLK_P: now also U8.45 (CSI_CLKN); no longer U8.44 (CSI_CLKP)
- net Earth: now also X5.14 (Pin_14)
- net GPIO30: no longer U8.60 (GPIO30)
- net GPIO39: now also X5.4 (Pin_4); no longer X5.5 (Pin_5)
- net GPIO40: now also X5.5 (Pin_5); no longer X5.6 (Pin_6)
- net GPIO41: now also X5.6 (Pin_6); no longer X5.7 (Pin_7)
- net GPIO42: now also X5.7 (Pin_7); no longer X5.8 (Pin_8)
- net GPIO43: now also X5.8 (Pin_8); no longer X5.9 (Pin_9)
- net GPIO44: now also X5.9 (Pin_9); no longer X5.10 (Pin_10)
- net SD_CLK: now also D6.7 (K6), U8.93 (GPIO50); no longer D6.9 (K8), U8.87 (GPIO45)
- net SD_CMD: now also U8.95 (GPIO52); no longer U8.88 (GPIO46)
- net SD_DATA0: now also U8.94 (GPIO51); no longer U8.89 (GPIO47)
- net SD_DATA1: now also D6.6 (K5), U8.92 (GPIO49); no longer D6.5 (K4), U8.90 (GPIO48)
- net SD_DATA2: now also D6.1 (K1), U8.97 (GPIO53); no longer D6.6 (K5), U8.92 (GPIO49)
- net SD_DATA3: now also D6.2 (K2), U8.98 (GPIO54); no longer D6.7 (K6), U8.93 (GPIO50)
- net USB_ESD_FS+: now also U5.4 (I/O2); no longer U5.6 (I/O1)
- net USB_ESD_FS-: now also U5.6 (I/O1); no longer U5.4 (I/O2)
- net USB_ESD_HS+: now also U4.4 (I/O2); no longer U4.6 (I/O1)
- net USB_ESD_HS-: now also U4.6 (I/O1); no longer U4.4 (I/O2)
- net USB_ESD_TTL+: now also U3.4 (I/O2); no longer U3.6 (I/O1)
- net USB_ESD_TTL-: now also U3.6 (I/O1); no longer U3.4 (I/O2)
- net USB_FS+: now also U5.3 (I/O2); no longer U5.1 (I/O1)
- net USB_FS-: now also U5.1 (I/O1); no longer U5.3 (I/O2)
- net USB_HS+: now also U4.3 (I/O2); no longer U4.1 (I/O1)
- net USB_HS-: now also U4.1 (I/O1); no longer U4.3 (I/O2)
- net USB_TTL+: now also U3.3 (I/O2); no longer U3.1 (I/O1)
- net USB_TTL-: now also U3.1 (I/O1); no longer U3.3 (I/O2)
- net at TP10.1, X9.9 (CD): now also D6.5 (K4); no longer D6.2 (K2)
- net GPIO31: no longer names the net of U8.61 (GPIO31)
- net GPIO31: no longer X5.2 (Pin_2)
- net GPIO32: no longer names the net of U8.63 (GPIO32)
- net GPIO32: no longer X5.3 (Pin_3)
- net GPIO33: no longer names the net of U8.64 (GPIO33)
- net GPIO33: no longer X5.4 (Pin_4)
- net GPIO51 renamed GPIO46
- net GPIO46: now also U8.88 (GPIO46); no longer U8.94 (GPIO51)
- net GPIO52 renamed GPIO47
- net GPIO47: now also U8.89 (GPIO47); no longer U8.95 (GPIO52)
- net GPIO53 renamed GPIO48
- net GPIO48: now also U8.90 (GPIO48); no longer U8.97 (GPIO53)
- removed net GPIO54: U8.98 (GPIO54), X5.14 (Pin_14)
- new net GPIO45: U8.87 (GPIO45), X5.10 (Pin_10)
- no-connect marks 40 -> 44
