File: ESP32-P4-dev-board.kicad_pcb (KiCad board)
At the start: 2 copper layers, 69.6 x 68.2 mm, 172 parts, among them Q1 SS8050, Q2 SS8050, SW1 KMR221GLFS, SW2 KMR221GLFS, SW3 KMR221GLFS, SW4 KMR221GLFS, U1 TLV62569DBV, U10 AP2127K-ADJTRG1, U11 AP2127K-ADJTRG1, U12 ESP-WROOM-02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

Commit message: трассировка и проверка завершены
Parts:
- C21, C28, C30, C39, C4, C5, C56, C60, R10, R3, R32, R33, R4, R5, R6, R9: moved to B.Cu
- X4, X5: footprint Connector_PinSocket_2.54mm:PinSocket_1x15_P2.54mm_Vertical -> Connector_PinSocket_1.27mm:PinSocket_1x15_P1.27mm_Vertical
- moved Y3 157.6 mm to (91.7, 61.5), turned to -90 degrees
- moved U10 153.7 mm to (88.2, 57.5), turned to -90 degrees
- moved U11 144.1 mm to (88.3, 78.4), turned to 90 degrees
- moved R36 143.2 mm to (95.9, 50.6)
- moved R30 141.4 mm to (90.9, 58.0), turned to 180 degrees
- moved R37 140.5 mm to (101.6, 50.6), turned to 180 degrees
- moved R43 139.9 mm to (97.8, 50.6)
- moved R44 139.8 mm to (99.7, 50.6), turned to 180 degrees
- moved R45 139.8 mm to (97.8, 55.1), turned to 180 degrees
- moved R46 139.6 mm to (99.8, 55.1)
- moved R28 139.2 mm to (90.9, 57.0), turned to 180 degrees
- moved R41 132.9 mm to (90.7, 73.7), turned to 90 degrees
- moved R10 131.3 mm to (93.6, 84.7), turned to 90 degrees
- moved R24 131.1 mm to (101.3, 61.5), turned to 90 degrees
- moved R25 131.0 mm to (103.3, 61.5), turned to 90 degrees
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Connections:
- D6 pad 1: +3.3V -> /SD_DATA2
- D6 pad 2: Net-(D6-K2) -> /SD_DATA3
- D6 pad 5: /SD_DATA1 -> Net-(D6-K4)
- D6 pad 6: /SD_DATA2 -> /SD_DATA1
- D6 pad 7: /SD_DATA3 -> /SD_CLK
- D6 pad 9: /SD_CLK -> +3.3V
- TP10 pad 1: Net-(D6-K2) -> Net-(D6-K4)
- U3 pad 1: USB_TTL+ -> USB_TTL-
- U3 pad 3: USB_TTL- -> USB_TTL+
- U3 pad 4: USB_ESD_TTL- -> USB_ESD_TTL+
- U3 pad 6: USB_ESD_TTL+ -> USB_ESD_TTL-
- U4 pad 1: USB_HS+ -> USB_HS-
- U4 pad 3: USB_HS- -> USB_HS+
- U4 pad 4: USB_ESD_HS- -> USB_ESD_HS+
- U4 pad 6: USB_ESD_HS+ -> USB_ESD_HS-
- U5 pad 1: USB_FS+ -> USB_FS-
- U5 pad 3: USB_FS- -> USB_FS+
- U5 pad 4: USB_ESD_FS- -> USB_ESD_FS+
- U5 pad 6: USB_ESD_FS+ -> USB_ESD_FS-
- U8 pad 44: CAM_CLK_P -> CAM_CLK_N
- U8 pad 45: CAM_CLK_N -> CAM_CLK_P
- U8 pad 60: /GPIO30 -> unconnected-(U8-GPIO30-Pad60)
- U8 pad 61: /GPIO31 -> unconnected-(U8-GPIO31-Pad61)
- U8 pad 63: /GPIO32 -> unconnected-(U8-GPIO32-Pad63)
- U8 pad 64: /GPIO33 -> unconnected-(U8-GPIO33-Pad64)
- U8 pad 87: /SD_CLK -> /GPIO45
- U8 pad 88: /SD_CMD -> /GPIO46
- U8 pad 89: /SD_DATA0 -> /GPIO47
- U8 pad 90: /SD_DATA1 -> /GPIO48
- U8 pad 92: /SD_DATA2 -> /SD_DATA1
- U8 pad 93: /SD_DATA3 -> /SD_CLK
- U8 pad 94: /GPIO51 -> /SD_DATA0
- U8 pad 95: /GPIO52 -> /SD_CMD
- U8 pad 97: /GPIO53 -> /SD_DATA2
- U8 pad 98: /GPIO54 -> /SD_DATA3
- X5 pad 10: /GPIO44 -> /GPIO45
- X5 pad 11: /GPIO51 -> /GPIO46
- X5 pad 12: /GPIO52 -> /GPIO47
- X5 pad 13: /GPIO53 -> /GPIO48
- X5 pad 14: /GPIO54 -> Earth
- X5 pad 2: /GPIO31 -> +3.3V
- X5 pad 3: /GPIO32 -> +3.3V
- X5 pad 4: /GPIO33 -> /GPIO39
- X5 pad 5: /GPIO39 -> /GPIO40
- X5 pad 6: /GPIO40 -> /GPIO41
- X5 pad 7: /GPIO41 -> /GPIO42
- X5 pad 8: /GPIO42 -> /GPIO43
- X5 pad 9: /GPIO43 -> /GPIO44
- X9 pad 9: Net-(D6-K2) -> Net-(D6-K4)
Routing:
- net I2C_SCL: track 0.00 -> 55.7 mm, vias 0 -> 3
- net CAM_EN: track 0.00 -> 52.3 mm, vias 0 -> 3
- net I2C_SDA: track 0.00 -> 51.6 mm, vias 0 -> 3
- net !RST: track 0.00 -> 41.5 mm, vias 0 -> 3
- net GPIO35_BOOTMODE: track 0.00 -> 38.5 mm, vias 0 -> 3
- net WS2812_DATA: track 0.00 -> 36.7 mm, vias 0 -> 2
- net /SD_DATA2: track 0.00 -> 34.6 mm, vias 0 -> 2
- net WIFI_EN: track 0.00 -> 34.3 mm, vias 0 -> 2
- net /SD_DATA3: track 0.00 -> 33.3 mm, vias 0 -> 2
- net /SD_CMD: track 0.00 -> 33.3 mm, vias 0 -> 2
- net /SD_CLK: track 0.00 -> 31.8 mm, vias 0 -> 2
- net DCDC_FB: track 0.00 -> 30.0 mm, vias 0 -> 2
- net +3.3V: track 0.00 -> 29.7 mm, vias 0 -> 53
- net /SD_DATA0: track 0.00 -> 27.7 mm, vias 0 -> 2
- net /SD_DATA1: track 0.00 -> 27.6 mm, vias 0 -> 2
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- added copper zone on F.Cu, net +1.5V
- added copper zone on F.Cu, net +2.8V
- added copper zone on In2.Cu, net +2.8V
- added copper zone on B.Cu, net +3.3V
- added copper zone on F.Cu, net +3.3V
- added copper zone on In2.Cu, net +3.3V
- added copper zone on B.Cu, net +5V
- added copper zone on F.Cu, net +5V
- added copper zone on In2.Cu, net +5V
- added copper zone on B.Cu, net 5V_HS
- added copper zone on F.Cu, net 5V_HS
- added copper zone on B.Cu, net 5V_TTL
- added copper zone on F.Cu, net 5V_TTL
- added copper zone on F.Cu, net ESP_VDD_HP
- added copper zone on In2.Cu, net ESP_VDD_HP
- added copper zone on B.Cu, net Earth
- added copper zone on F.Cu, net Earth
- added copper zone on In1.Cu, net Earth
- added copper zone on F.Cu, net Net-(C65-Pad1)
- added copper zone on F.Cu, net Net-(U1-SW)
- added copper zone on F.Cu, net Net-(U2-SW)
- added copper zone on F.Cu, net VDDMIPI
- added copper zone on In2.Cu, net VDDMIPI
- added copper zone on B.Cu, net VDDPST
Other:
- board size 69.6 x 68.2 mm -> 68.2 x 43.3 mm
- copper layers 2 -> 4

Commit message: Rev 0 ready
Parts:
- added kibuzzard-6926A799: G***, kibuzzard-6926A799, F.Cu at (114.5, 57.6)
Routing:
- net Earth: vias 215 -> 236
- net CAM_EN: vias 3 -> 5
Other:
- board text added: "+3.3"
- board text added: "BOOT"
- board text added: "ESP32"
- board text added: "GND"
- board text added: "GPIO10"
- board text added: "GPIO11"
- board text added: "GPIO12"
- board text added: "GPIO13"
- board text added: "GPIO14"
- board text added: "GPIO15"
- board text added: "GPIO20"
- board text added: "GPIO23"
- board text added: "GPIO30"
- board text added: "GPIO39"
- board text added: "GPIO40"
- board text added: "GPIO41"
- board text added: "GPIO42"
- board text added: "GPIO43"
- board text added: "GPIO44"
- board text added: "GPIO45"
- board text added: "GPIO46"
- board text added: "GPIO47"
- board text added: "GPIO48"
- board text added: "GPIO6"
- board text added: "GPIO7"
- board text added: "GPIO8"
- board text added: "GPIO9"
- board text added: "RST"
- board text added: "RX"
- board text added: "SCL"
- board text added: "SDA"
- board text added: "TX"
- board text added: "USB-FS"
- board text added: "USB-HS"
- board text added: "USB-TTL"
- board text added: "WIFI"
- board text added: "by @madjogger"
